Commit message: fixed mini-cheetah.urdf

File: rsc/minicheetah/mini-cheetah.urdf (robot description, URDF)
Before this commit: robot mini_cheetah, 13 links, 12 joints
Links:
- added link toe_fl, mass 0.0; collision sphere radius=0.02; visual sphere radius=0.02
- added link toe_fr, mass 0.0; collision sphere radius=0.02; visual sphere radius=0.02
- added link toe_hl, mass 0.0; collision sphere radius=0.02; visual sphere radius=0.02
- added link toe_hr, mass 0.0; collision sphere radius=0.02; visual sphere radius=0.02
- link abduct_fl: geometry collision cylinder length=0.022 radius=0.048; visual mesh filename=meshes/mini_abad.obj
- link abduct_fr: geometry collision cylinder length=0.022 radius=0.048; visual mesh filename=meshes/mini_abad.obj
- link abduct_hl: geometry collision cylinder length=0.022 radius=0.048; visual mesh filename=meshes/mini_abad.obj
- link abduct_hr: geometry collision cylinder length=0.022 radius=0.048; visual mesh filename=meshes/mini_abad.obj
- link body: mass 3.3 -> 5.868; geometry collision box size=0.244 0.18 0.09; visual mesh filename=meshes/mini_body.obj
- link shank_fl: geometry collision box size=0.016 0.016 0.18; visual mesh filename=meshes/mini_lower_link.obj
- link shank_fr: geometry collision box size=0.016 0.016 0.18; visual mesh filename=meshes/mini_lower_link.obj
- link shank_hl: geometry collision box size=0.016 0.016 0.18; visual mesh filename=meshes/mini_lower_link.obj
- link shank_hr: geometry collision box size=0.016 0.016 0.18; visual mesh filename=meshes/mini_lower_link.obj
- link thigh_fl: geometry collision box size=0.025 0.025 0.16; visual mesh filename=meshes/mini_upper_link.obj
- link thigh_fr: geometry collision box size=0.025 0.025 0.16; visual mesh filename=meshes/mini_upper_link.obj
- link thigh_hl: geometry collision box size=0.025 0.025 0.16; visual mesh filename=meshes/mini_upper_link.obj
- link thigh_hr: geometry collision box size=0.025 0.025 0.16; visual mesh filename=meshes/mini_upper_link.obj
Joints:
- added joint toe_fl_joint: type fixed, parent shank_fl, child toe_fl, origin xyz=0 0 -0.18
- added joint toe_fr_joint: type fixed, parent shank_fr, child toe_fr, origin xyz=0 0 -0.18
- added joint toe_hl_joint: type fixed, parent shank_hl, child toe_hl, origin xyz=0 0 -0.18
- added joint toe_hr_joint: type fixed, parent shank_hr, child toe_hr, origin xyz=0 0 -0.18
- joint abduct_fl_to_thigh_fl_j: limit (none) -> lower=-4.712388 upper=4.712388 effort=18 velocity=40; type continuous -> revolute
- joint abduct_fr_to_thigh_fr_j: limit (none) -> lower=-4.712388 upper=4.712388 effort=18 velocity=40; type continuous -> revolute
- joint abduct_hl_to_thigh_hl_j: limit (none) -> lower=-4.712388 upper=4.712388 effort=18 velocity=40; type continuous -> revolute
- joint abduct_hr_to_thigh_hr_j: limit (none) -> lower=-4.712388 upper=4.712388 effort=18 velocity=40; type continuous -> revolute
- joint thigh_fl_to_knee_fl_j: limit (none) -> lower=-2.705259778 upper=2.705259778 effort=11.6 velocity=40; type continuous -> revolute
- joint thigh_fr_to_knee_fr_j: limit (none) -> lower=-2.705259778 upper=2.705259778 effort=11.6 velocity=40; type continuous -> revolute
- joint thigh_hl_to_knee_hl_j: limit (none) -> lower=-2.705259778 upper=2.705259778 effort=11.6 velocity=40; type continuous -> revolute
- joint thigh_hr_to_knee_hr_j: limit (none) -> lower=-2.705259778 upper=2.705259778 effort=11.6 velocity=40; type continuous -> revolute
- joint torso_to_abduct_fl_j: limit (none) -> lower=-2.094395102 upper=2.094395102 effort=18 velocity=40; type continuous -> revolute
- joint torso_to_abduct_fr_j: limit (none) -> lower=-2.094395102 upper=2.094395102 effort=18 velocity=40; type continuous -> revolute
- joint torso_to_abduct_hl_j: limit (none) -> lower=-2.094395102 upper=2.094395102 effort=18 velocity=40; type continuous -> revolute
- joint torso_to_abduct_hr_j: limit (none) -> lower=-2.094395102 upper=2.094395102 effort=18 velocity=40; origin xyz=0.2 -0.049 0.0 rpy=0 0 0 -> xyz=-0.2 -0.049 0.0 rpy=0 0 0; type continuous -> revolute
