Commit message: feat: Position based deeploco update

File: rsc/raibo_arm/urdf/raibo_arm.urdf (robot description, URDF)
Before this commit: robot raibo_arm, 28 links, 27 joints
Links:
- link LF_FOOT: geometry collision sphere radius=0.0295; visual mesh filename=LF_FOOT.STL
- link LH_FOOT: geometry collision sphere radius=0.0295; visual mesh filename=LH_FOOT.STL
- link RF_FOOT: geometry collision sphere radius=0.0295; visual mesh filename=RF_FOOT.STL
- link RH_FOOT: geometry collision sphere radius=0.0295; visual mesh filename=RH_FOOT.STL

File: rsc/raibot/urdf/raibot_simplified.urdf (robot description, URDF)
Before this commit: robot raibot, 17 links, 16 joints
Links:
- link LF_SHANK: geometry collision box size=0.1711 0.020 0.0253; visual mesh filename=LF_SHANK.STL
- link LF_THIGH: geometry collision cylinder length=0.053 radius=0.0265; visual mesh filename=LF_THIGH.STL
- link LH_SHANK: geometry collision box size=0.1711 0.020 0.0253; visual mesh filename=LH_SHANK.STL
- link LH_THIGH: geometry collision cylinder length=0.053 radius=0.0265; visual mesh filename=LH_THIGH.STL
- link RF_SHANK: geometry collision box size=0.1711 0.020 0.0253; visual mesh filename=RF_SHANK.STL
- link RF_THIGH: geometry collision cylinder length=0.053 radius=0.0265; visual mesh filename=RF_THIGH.STL
- link RH_SHANK: geometry collision box size=0.1711 0.020 0.0253; visual mesh filename=RH_SHANK.STL
- link RH_THIGH: geometry collision cylinder length=0.053 radius=0.0265; visual mesh filename=RH_THIGH.STL
