Commit message: Temp

File: default_controller_demo/rsc/raibot/urdf/raibot_simplified_manipulator.urdf (robot description, URDF)
Before this commit: robot raibot, 17 links, 16 joints
Links:
- added link arm, mass 0.1; collision box size=0.1 0.04 0.3; visual box size=0.1 0.04 0.3
- link LF_SHANK: geometry collision box size=0.1711 0.020 0.0253; visual mesh filename=LF_SHANK.STL
- link LF_THIGH: geometry collision cylinder length=0.053 radius=0.0265; visual mesh filename=LF_THIGH.STL
- link LH_SHANK: geometry collision box size=0.1711 0.020 0.0253; visual mesh filename=LH_SHANK.STL
- link LH_THIGH: geometry collision cylinder length=0.053 radius=0.0265; visual mesh filename=LH_THIGH.STL
- link RF_SHANK: geometry collision box size=0.1711 0.020 0.0253; visual mesh filename=RF_SHANK.STL
- link RF_THIGH: geometry collision cylinder length=0.053 radius=0.0265; visual mesh filename=RF_THIGH.STL
- link RH_SHANK: geometry collision box size=0.1711 0.020 0.0253; visual mesh filename=RH_SHANK.STL
- link RH_THIGH: geometry collision cylinder length=0.053 radius=0.0265; visual mesh filename=RH_THIGH.STL
- link base: geometry collision box size=0.7104 0.276 0.120; visual mesh filename=base.STL
Joints:
- added joint base_arm: type fixed, parent base, child LF_HIP, origin xyz=0.3072 0.0 -0.05 rpy=0 0 0, axis 1 0 0

File: rsc/raibot/urdf/raibot_simplified_manipulator.urdf (robot description, URDF)
Before this commit: robot raibot, 17 links, 16 joints
Links:
- added link arm, mass 0.1; collision box size=0.1 0.04 0.3; visual box size=0.1 0.04 0.3
- link LF_SHANK: geometry collision box size=0.1711 0.020 0.0253; visual mesh filename=LF_SHANK.STL
- link LF_THIGH: geometry collision cylinder length=0.053 radius=0.0265; visual mesh filename=LF_THIGH.STL
- link LH_SHANK: geometry collision box size=0.1711 0.020 0.0253; visual mesh filename=LH_SHANK.STL
- link LH_THIGH: geometry collision cylinder length=0.053 radius=0.0265; visual mesh filename=LH_THIGH.STL
- link RF_SHANK: geometry collision box size=0.1711 0.020 0.0253; visual mesh filename=RF_SHANK.STL
- link RF_THIGH: geometry collision cylinder length=0.053 radius=0.0265; visual mesh filename=RF_THIGH.STL
- link RH_SHANK: geometry collision box size=0.1711 0.020 0.0253; visual mesh filename=RH_SHANK.STL
- link RH_THIGH: geometry collision cylinder length=0.053 radius=0.0265; visual mesh filename=RH_THIGH.STL
- link base: geometry collision box size=0.1 0.1 0.120; visual mesh filename=base.STL
