Commit message: Feat: add raibo cam sensor

File: examples/examples/rsc/raibo2_arm/urdf/raibo2_arm.urdf (robot description, URDF)
Before this commit: robot raibo2_arm, 8 links, 7 joints
Links:
- link base_link: geometry collision mesh filename=../meshes/base_link.obj; visual mesh filename=../meshes/base_link.STL
- link link1: geometry collision mesh filename=../meshes/link1.obj; visual mesh filename=../meshes/link1.STL
- link link2: mass 0.8582 -> 0.84768; geometry collision mesh filename=../meshes/link2.obj; visual mesh filename=../meshes/link2.STL
- link link3: mass 0.34252 -> 0.300280421855983; geometry collision mesh filename=../meshes/link3.obj; visual mesh filename=../meshes/link3.STL
- link link4: mass 0.32249 -> 0.322493892765723; geometry collision mesh filename=../meshes/link4.obj; visual mesh filename=../meshes/link4.STL
- link link5: mass 0.27079 -> 0.270793262476203; geometry collision mesh filename=../meshes/link5.obj; visual mesh filename=../meshes/link5.STL
- link link6: mass 0.026017 -> 0.00616895938082152; geometry collision mesh filename=../meshes/link6.obj; visual mesh filename=../meshes/link6.STL
Joints:
- joint joint1: axis 0 0 1 -> 0 0 -1; limit lower=-6.28 upper=6.28 effort=80 velocity=20 -> lower=-3.28 upper=3.28 effort=80 velocity=20; origin xyz=-0.14165 -0.39992 -0.29982 rpy=-0.37519 0.40075 -2.8051 -> xyz=0 6.0353E-05 0.066545 rpy=0 0 -0.45605
- joint joint2: axis 0 0 1 -> 0 0 -1; limit lower=-6.28 upper=6.28 effort=80 velocity=20 -> lower=-3.28 upper=3.28 effort=80 velocity=20; origin xyz=-5.52E-05 0.0039996 0.053 rpy=-1.5708 0.97319 0.013801 -> xyz=0 -0.007 0.053 rpy=1.5708 -0.19845 0
- joint joint3: limit lower=-2.5 upper=0.5 effort=80 velocity=20 -> lower=-1.8 upper=0.4 effort=80 velocity=20; origin xyz=0.31352 -0.064094 0.08565 rpy=3.1416 0 -1.1678 -> xyz=-0.22627 0.22627 0.08265 rpy=3.1416 0 -2.1523
- joint joint4: axis 0 0 1 -> 0 0 -1; limit lower=-6.28 upper=6.28 effort=40 velocity=20 -> lower=-3.28 upper=3.28 effort=40 velocity=20; origin xyz=0.07 0 0 rpy=1.5708 1.5397 1.5708 -> xyz=-0.070002 0 0 rpy=1.5708 1.063 -1.5708
- joint joint5: limit lower=-2.5 upper=2.5 effort=40 velocity=20 -> lower=-1.5 upper=1.5 effort=40 velocity=20; origin xyz=-0.02768 -0.0042217 0.359 rpy=1.5708 -1.3841 -1.4194 -> xyz=0.0076283 -0.026945 0.359 rpy=-1.5708 1.3723 -2.8657
- joint joint6: axis 0 0 1 -> 0 0 -1; limit lower=-6.28 upper=6.28 effort=40 velocity=10 -> lower=-3.28 upper=3.28 effort=40 velocity=20; origin xyz=0.086577 0.01576 -0.028 rpy=-1.5708 -1.1675 -1.3907 -> xyz=-0.088002 0 -0.028004 rpy=-1.5708 0.63873 1.5708

File: rsc/raibot/urdf/raibot_simplified.urdf (robot description, URDF)
Before this commit: robot raibot, 18 links, 17 joints
Links:
- added link depth_camera_front_camera, mass 0.16043; visual mesh filename=sensors/depth_camera.dae scale=1.0 1.0 1.0
- added link depth_camera_front_camera_parent
- added link depth_camera_front_color_frame
- added link depth_camera_front_color_optical_frame
- added link depth_camera_front_depth_optical_frame
- added link wide_angle_camera_front_camera, mass 0.287; visual mesh filename=sensors/wide_angle_camera.dae scale=1.0 1.0 1.0
- added link wide_angle_camera_front_camera_parent
Joints:
- added joint depth_camera_front_camera_parent_to_color_frame: type fixed, parent depth_camera_front_camera_parent, child depth_camera_front_color_frame, origin xyz=0 0.015 0 rpy=0 0 0
- added joint depth_camera_front_camera_parent_to_depth_optical_frame: type fixed, parent depth_camera_front_camera_parent, child depth_camera_front_depth_optical_frame, origin xyz=0.0 0.0 0.0 rpy=-1.57079632679 0.0 -1.57079632679
- added joint depth_camera_front_camera_to_camera_parent: type fixed, parent depth_camera_front_camera, child depth_camera_front_camera_parent, origin xyz=0.0255 0.0175 0.0 rpy=0.0 0.0 0.0
- added joint depth_camera_front_color_frame_to_color_optical_frame: type fixed, parent depth_camera_front_color_frame, child depth_camera_front_color_optical_frame, origin xyz=0.0 0.0 0.0 rpy=-1.57079632679 0.0 -1.57079632679
- added joint face_front_to_depth_camera_front_camera: type fixed, parent arm_link, child depth_camera_front_camera, origin xyz=-0.05 0.0 0.1 rpy=0.0 -0.1 0
- added joint face_front_to_wide_angle_camera_front_camera: type fixed, parent arm_link, child wide_angle_camera_front_camera, origin xyz=0.09850 0.0 0.01497 rpy=0 0 0
- added joint wide_angle_camera_front_camera_to_camera_parent: type fixed, parent wide_angle_camera_front_camera, child wide_angle_camera_front_camera_parent, origin xyz=0.0 0.0 0.0 rpy=-1.57079632679 0.0 -1.57079632679
