Commit message: working version. need more tuning

File: rsc/raibot/urdf/raibot_simplified.urdf (robot description, URDF)
Before this commit: robot raibot, 17 links, 16 joints
Links:
- link LF_SHANK: geometry collision box size=0.1311 0.020 0.0253; visual mesh filename=LF_SHANK.STL
- link LH_SHANK: geometry collision box size=0.1311 0.020 0.0253; visual mesh filename=LH_SHANK.STL
- link RF_SHANK: geometry collision box size=0.1311 0.020 0.0253; visual mesh filename=RF_SHANK.STL
- link RH_SHANK: geometry collision box size=0.1311 0.020 0.0253; visual mesh filename=RH_SHANK.STL

Commit message: Feat: Sigmoid, add damping, one hot vector, object ori

File: rsc/raibot/urdf/raibot_simplified.urdf (robot description, URDF)
Before this commit: robot raibot, 17 links, 16 joints
Links:
- link LF_SHANK: geometry collision box size=0.1711 0.020 0.0253; visual mesh filename=LF_SHANK.STL
- link LF_THIGH: geometry collision cylinder length=0.053 radius=0.0265; visual mesh filename=LF_THIGH.STL
- link LH_SHANK: geometry collision box size=0.1711 0.020 0.0253; visual mesh filename=LH_SHANK.STL
- link LH_THIGH: geometry collision cylinder length=0.053 radius=0.0265; visual mesh filename=LH_THIGH.STL
- link RF_SHANK: geometry collision box size=0.1711 0.020 0.0253; visual mesh filename=RF_SHANK.STL
- link RF_THIGH: geometry collision cylinder length=0.053 radius=0.0265; visual mesh filename=RF_THIGH.STL
- link RH_SHANK: geometry collision box size=0.1711 0.020 0.0253; visual mesh filename=RH_SHANK.STL
- link RH_THIGH: geometry collision cylinder length=0.053 radius=0.0265; visual mesh filename=RH_THIGH.STL

Commit message: Feat: collision body fixed, exteroceptive info added

File: rsc/raibot/urdf/raibot_simplified.urdf (robot description, URDF)
Before this commit: robot raibot, 17 links, 16 joints
Links:
- added link arm_link, mass 0.001; collision cylinder length=0.05 radius=0.05; visual box size=0.001 0.001 0.001
- link base: geometry collision box size=0.7104 0.276 0.120; visual mesh filename=base.STL
Joints:
- added joint arm: type fixed, parent base, child arm_link, origin xyz=0.6 0 -0.2 rpy=0 0 0

Commit message: feat: remove arm & target to ee changed

File: rsc/raibot/urdf/raibot_simplified.urdf (robot description, URDF)
Before this commit: robot raibot, 18 links, 17 joints
Links:
- link LF_HIP: geometry collision cylinder length=0.06 radius=0.047; collision cylinder length=0.08 radius=0.047
- link LF_THIGH: geometry collision box size=0.14 0.03 0.0253; collision cylinder length=0.053 radius=0.0265
- link LH_HIP: geometry collision cylinder length=0.06 radius=0.047; collision cylinder length=0.08 radius=0.047
- link LH_THIGH: geometry collision box size=0.14 0.03 0.0253; collision cylinder length=0.053 radius=0.0265
- link RF_HIP: geometry collision cylinder length=0.06 radius=0.047; collision cylinder length=0.08 radius=0.047
- link RF_THIGH: geometry collision box size=0.14 0.03 0.0253; collision cylinder length=0.053 radius=0.0265
- link RH_HIP: geometry collision cylinder length=0.06 radius=0.047; collision cylinder length=0.08 radius=0.047
- link RH_THIGH: geometry collision box size=0.14 0.03 0.0253; collision cylinder length=0.053 radius=0.0265
- link arm_link: geometry visual box size=0.01 0.01 0.01
- link base: geometry collision box size=0.48 0.27 0.120; visual mesh filename=base.STL
Joints:
- joint arm: origin xyz=0.6 0 -0.2 rpy=0 0 0 -> xyz=0.35 0 -0.03 rpy=0 0 0

Commit message: feat: get camera pose feat: get camera image feat: office environment generation in Unreal

File: rsc/raibot/urdf/raibot_simplified.urdf (robot description, URDF)
Before this commit: robot raibot, 18 links, 17 joints
Links:
- removed link arm_link
- link LF_HIP: geometry visual mesh filename=LF_HIP.STL
- link LF_SHANK: geometry collision box size=0.1311 0.020 0.0253; visual mesh filename=LF_SHANK.STL
- link LF_THIGH: geometry collision capsule length=0.053 radius=0.0265; visual mesh filename=LF_THIGH.STL
- link LH_HIP: geometry visual mesh filename=LH_HIP.STL
- link LH_SHANK: geometry collision box size=0.1311 0.020 0.0253; visual mesh filename=LH_SHANK.STL
- link LH_THIGH: geometry collision capsule length=0.053 radius=0.0265; visual mesh filename=LH_THIGH.STL
- link RF_HIP: geometry visual mesh filename=RF_HIP.STL
- link RF_SHANK: geometry collision box size=0.1311 0.020 0.0253; visual mesh filename=RF_SHANK.STL
- link RF_THIGH: geometry collision capsule length=0.053 radius=0.0265; visual mesh filename=RF_THIGH.STL
- link RH_HIP: geometry visual mesh filename=RH_HIP.STL
- link RH_SHANK: geometry collision box size=0.1311 0.020 0.0253; visual mesh filename=RH_SHANK.STL
- link RH_THIGH: geometry collision capsule length=0.053 radius=0.0265; visual mesh filename=RH_THIGH.STL
- link base: geometry collision box size=0.36 0.13 0.120; visual mesh filename=base.STL
Joints:
- removed joint arm
